File: PCB-KiCad/ESP32j1mmb/ESP32j1mmb.kicad_pcb (KiCad board)
At the start: 2 copper layers, 34 x 45.5 mm, 11 parts, among them J1 FTDI+DTR, J2 Left, J3 Left, U1 ESP32-WROOM-32, U2 AP1117-33

Commit message: Experimented with silkscreen issues.. updated README.
Parts:
- J1: value FTDI+DTR -> GND - FTDI
Other:
- board text added: "GND - FTDI"
- board text added: "RTS"
Changed lines of the file:
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@@
 		(allow_soldermask_bridges_in_footprints no)
 		(pcbplotparams
-			(layerselection 0x00010fc_ffffffff)
+			(layerselection 0x00210fc_ffffffff)
 			(plot_on_all_layers_selection 0x0000000_00000000)
 			(disableapertmacros no)
@@
 		(tags "resistor handsolder")
 		(property "Reference" "R1"
-			(at 0 -1.43 360)
+			(at 0 -1.43 0)
 			(layer "F.SilkS")
 			(hide yes)
@@
 		)
 		(fp_text user "${REFERENCE}"
-			(at 0 0 360)
+			(at 0 0 0)
 			(layer "F.Fab")
 			(effects
@@
 		(tags "capacitor handsolder")
 		(property "Reference" "C2"
-			(at 0 -1.43 270)
+			(at 0 -1.43 -90)
 			(layer "F.SilkS")
 			(hide yes)
@@
 		)
 		(property "Value" "100n"
-			(at -0.5 -1.5 270)
+			(at -0.5 -1.5 -90)
 			(layer "F.SilkS")
 			(effects
@@
 		)
 		(fp_text user "${REFERENCE}"
-			(at 0 0 270)
+			(at 0 0 -90)
 			(layer "F.Fab")
 			(effects
@@
 			)
 		)
-		(property "Value" "FTDI+DTR"
-			(at -2.5 3.7 180)
+		(property "Value" "GND -  FTDI"
+			(at -2.059992 9.057335 180)
 			(layer "F.SilkS")
+			(hide yes)
 			(effects
 				(font
@@
 		(tags "resistor handsolder")
 		(property "Reference" "R2"
-			(at 0 -1.43 360)
+			(at 0 -1.43 0)
 			(layer "F.SilkS")
 			(hide yes)
@@
 		)
 		(fp_text user "${REFERENCE}"
-			(at 0 0 360)
+			(at 0 0 0)
 			(layer "F.Fab")
 			(effects
@@
 		(tags "capacitor handsolder")
 		(property "Reference" "C1"
-			(at 0.5 1.5 270)
+			(at 0.5 1.5 -90)
 			(layer "F.SilkS")
 			(hide yes)
@@
 		)
 		(property "Value" "10u"
-			(at 0 1.43 270)
+			(at 0 1.43 -90)
 			(layer "F.SilkS")
 			(effects
@@
 		)
 		(fp_text user "${REFERENCE}"
-			(at 0 0 270)
+			(at 0 0 -90)
 			(layer "F.Fab")
 			(effects
@@
 		(layer "F.SilkS")
 		(effects
+			(font
+				(size 1 1)
+				(thickness 0.1)
+			)
+			(justify left bottom)
+		)
+	)
+	(gr_text "GND -  FTDI"
+		(at 83.709935 134.017286 0)
+		(layer "F.SilkS")
+		(effects
+			(font
+				(size 1 1)
+				(thickness 0.1)
+			)
+			(justify left bottom)
+		)
+	)
+	(gr_text "RTS"
+		(at 81 134 0)
+		(layer "F.SilkS")
+		(effects
